Commit message: Integrated the bot with gazebo in an empty world

File: urdf/turtlebot.urdf (robot description, URDF)
Before this commit: robot turtlebot, 59 links, 58 joints
Links:
- link arm_base_link: geometry collision mesh filename=package://turtlebot/meshes/PincherBase.stl scale=1.0 1.0 1.0; visual mesh filename=package://turtlebot/meshes/PincherBase.stl scale=1.0 1.0 1.0
- link arm_bicep_link: geometry collision mesh filename=package://turtlebot/meshes/PincherBicep.stl scale=1.0 1.0 1.0; visual mesh filename=package://turtlebot/meshes/PincherBicep.stl scale=1.0 1.0 1.0
- link arm_forearm_link: geometry collision mesh filename=package://turtlebot/meshes/PincherForeArm.stl scale=1.0 1.0 1.0; visual mesh filename=package://turtlebot/meshes/PincherForeArm.stl scale=1.0 1.0 1.0
- link arm_shoulder_pan_link: geometry collision mesh filename=package://turtlebot/meshes/F2Bracket.stl scale=1.0 1.0 1.0; visual mesh filename=package://turtlebot/meshes/F2Bracket.stl scale=1.0 1.0 1.0
- link arm_wrist_flex_link: geometry collision mesh filename=package://turtlebot/meshes/PincherWristGripper.stl scale=1.0 1.0 1.0; visual mesh filename=package://turtlebot/meshes/PincherWristGripper.stl scale=1.0 1.0 1.0
- link gripper_active2_link: geometry collision mesh filename=package://turtlebot/meshes/PincherFinger.stl scale=1.0 1.0 1.0; visual mesh filename=package://turtlebot/meshes/PincherFinger.stl scale=1.0 1.0 1.0
- link gripper_active_link: geometry collision mesh filename=package://turtlebot/meshes/PincherFinger.stl scale=1.0 1.0 1.0; visual mesh filename=package://turtlebot/meshes/PincherFinger.stl scale=1.0 1.0 1.0
